File: hardware/ISL29125 Breakout.brd (EAGLE design)
At the start: 17.8 x 16.5 mm, 16 parts, among them U1 ISL29125

Commit message: v01, revised after review, ready for protos
Parts:
- removed LOGO1: SFE_LOGO_NAME_FLAME.1_INCH, SparkFun-Aesthetics:SFE_LOGO_NAME_FLAME_.1
- added LOGO2: SFE_LOGO_FLAME.2_INCH, SparkFun-Aesthetics:SFE_LOGO_FLAME_.2
- added SJ2: (no value), SparkFun-Passives:SJ_3
- moved LOGO3 8.17 mm to (10.2, 14.0)
- moved C1 1.90 mm to (3.81, 8.26)
- moved C2 1.90 mm to (3.81, 10.2)
Connections:
- new net N$3: R2.2, SJ2.3
- new net N$4: R3.2, SJ2.1
- net 3.3V: now also SJ2.2; no longer R2.2, R3.2
Routing:
- net 3.3V: track 21.8 -> 27.3 mm, vias 1 -> 3
- net N$4: track 0.00 -> 4.16 mm, vias 0 -> 1
- net N$3: track 0.00 -> 3.78 mm, vias 0 -> 1
- net GND: track 13.4 -> 12.0 mm
Other:
- board text added: "I2C: 0x44"
- board text added: "pullups"

Commit message: hardware ready for reds, v10
Parts:
- moved LOGO4 0.25 mm to (11.3, 11.6)
Other:
- board text added: "v10"
- board text removed: "pullups"
- board text removed: "v01"
Changed lines of the file:
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@@
 <layer number="27" name="tValues" color="7" fill="1" visible="no" active="yes"/>
 <layer number="28" name="bValues" color="7" fill="1" visible="no" active="yes"/>
-<layer number="29" name="tStop" color="7" fill="3" visible="no" active="yes"/>
+<layer number="29" name="tStop" color="7" fill="3" visible="yes" active="yes"/>
 <layer number="30" name="bStop" color="7" fill="6" visible="no" active="yes"/>
-<layer number="31" name="tCream" color="7" fill="4" visible="no" active="yes"/>
+<layer number="31" name="tCream" color="7" fill="4" visible="yes" active="yes"/>
 <layer number="32" name="bCream" color="7" fill="5" visible="no" active="yes"/>
 <layer number="33" name="tFinish" color="6" fill="3" visible="no" active="yes"/>
@@
 <layer number="39" name="tKeepout" color="4" fill="11" visible="no" active="yes"/>
 <layer number="40" name="bKeepout" color="1" fill="11" visible="no" active="yes"/>
-<layer number="41" name="tRestrict" color="4" fill="10" visible="no" active="yes"/>
+<layer number="41" name="tRestrict" color="4" fill="10" visible="yes" active="yes"/>
 <layer number="42" name="bRestrict" color="1" fill="10" visible="no" active="yes"/>
 <layer number="43" name="vRestrict" color="2" fill="10" visible="no" active="yes"/>
@@
 <text x="14.478" y="2.794" size="1.016" layer="21" font="vector" ratio="15" rot="R90">!INT</text>
 <text x="8.128" y="12.954" size="1.016" layer="22" font="vector" ratio="15" rot="SMR270">ISL29125</text>
-<text x="17.018" y="3.937" size="1.016" layer="21" font="vector" ratio="15" rot="R90">ISL29125</text>
 <text x="9.525" y="10.541" size="1.016" layer="22" font="vector" ratio="15" rot="SMR270">RGB</text>
 <text x="10.795" y="11.811" size="1.016" layer="22" font="vector" ratio="15" rot="SMR270">Sensor</text>
-<text x="16.891" y="3.429" size="1.016" layer="16" font="vector" ratio="15" rot="SMR270">v01</text>
+<text x="16.891" y="3.429" size="1.016" layer="16" font="vector" ratio="15" rot="SMR270">v10</text>
 <text x="-2.159" y="-22.225" size="1.778" layer="25" font="vector" ratio="15">Jordan McConnell</text>
 <text x="3.302" y="2.794" size="1.016" layer="22" font="vector" ratio="15" rot="SMR270" align="top-right">GND</text>
@@
 <text x="10.922" y="2.794" size="1.016" layer="22" font="vector" ratio="15" rot="SMR270" align="top-right">SCL</text>
 <text x="13.462" y="2.794" size="1.016" layer="22" font="vector" ratio="15" rot="SMR270" align="top-right">!INT</text>
-<text x="14.478" y="7.112" size="0.254" layer="22" font="vector" ratio="15" rot="SMR270">pullups</text>
 <text x="15.621" y="9.144" size="0.6096" layer="22" font="vector" ratio="15" rot="SMR270">SDA</text>
 <text x="17.399" y="5.08" size="0.6096" layer="22" font="vector" ratio="15" rot="SMR270">SCL</text>
 <text x="16.637" y="5.08" size="0.6096" layer="22" font="vector" ratio="15" rot="SMR270">3.3V</text>
 <text x="1.524" y="5.207" size="0.6096" layer="22" font="vector" ratio="15" rot="SMR270">I2C: 0x44</text>
+<text x="1.524" y="4.826" size="1.016" layer="21" font="vector" ratio="15" rot="R90">ISL29125</text>
+<rectangle x1="7.874" y1="8.128" x2="8.89" y2="8.255" layer="41"/>
 </plain>
 <attributes>
@@
 <element name="STANDOFF1" library="SparkFun-Electromechanical" package="STAND-OFF" value="STAND-OFF" x="2.54" y="13.97"/>
 <element name="STANDOFF2" library="SparkFun-Electromechanical" package="STAND-OFF" value="STAND-OFF" x="15.24" y="13.97"/>
-<element name="LOGO4" library="SparkFun-Aesthetics" package="SFE_LOGO_FLAME_.2" value="SFE_LOGO_FLAME.2_INCH" x="11.557" y="11.557" rot="R90"/>
+<element name="LOGO4" library="SparkFun-Aesthetics" package="SFE_LOGO_FLAME_.2" value="SFE_LOGO_FLAME.2_INCH" x="11.303" y="11.557" rot="R90"/>
 <element name="SJ2" library="SparkFun-Passives" package="SJ_3" value="" x="16.256" y="6.35" rot="MR0"/>
 <element name="LOGO2" library="SparkFun-Aesthetics" package="SFE_LOGO_FLAME_.2" value="SFE_LOGO_FLAME.2_INCH" x="6.477" y="11.303" rot="SMR270"/>
@@
 <wire x1="14.82" y1="10.16" x2="15.748" y2="10.16" width="0.2032" layer="1"/>
 <wire x1="15.748" y1="10.16" x2="16.256" y2="9.652" width="0.2032" layer="1"/>
-<wire x1="16.256" y1="9.652" x2="16.256" y2="9.144" width="0.2032" layer="1"/>
-<via x="16.256" y="9.144" extent="1-16" drill="0.508"/>
+<via x="16.256" y="9.652" extent="1-16" drill="0.508"/>
 <wire x1="16.256" y1="6.35" x2="16.256" y2="4.064" width="0.2032" layer="16"/>
 <wire x1="16.256" y1="4.064" x2="15.367" y2="3.175" width="0.2032" layer="16"/>
@@
 <wire x1="10.16" y1="3.81" x2="8.89" y2="3.81" width="0.2032" layer="16"/>
 <wire x1="8.89" y1="3.81" x2="6.35" y2="1.27" width="0.2032" layer="16"/>
-<wire x1="16.256" y1="9.144" x2="16.256" y2="6.35" width="0.2032" layer="16"/>
 <wire x1="16.256" y1="6.35" x2="17.272" y2="6.35" width="0.2032" layer="16"/>
 <wire x1="15.24" y1="6.35" x2="15.875" y2="6.35" width="0.2032" layer="16"/>
 <wire x1="15.875" y1="6.35" x2="16.256" y2="6.35" width="0.2032" layer="16"/>
+<wire x1="16.256" y1="9.652" x2="16.256" y2="9.271" width="0.2032" layer="16"/>
+<wire x1="16.256" y1="9.271" x2="15.748" y2="8.763" width="0.2032" layer="16"/>
+<wire x1="15.748" y1="8.763" x2="15.748" y2="7.747" width="0.2032" layer="16"/>
+<wire x1="15.748" y1="7.747" x2="16.256" y2="7.239" width="0.2032" layer="16"/>
+<wire x1="16.256" y1="7.239" x2="16.256" y2="6.35" width="0.2032" layer="16"/>
 </signal>
 <signal name="!INT">
@@
 <contactref element="R3" pad="2"/>
 <contactref element="SJ2" pad="1"/>
-<wire x1="14.82" y1="8.255" x2="17.018" y2="8.255" width="0.2032" layer="1"/>
-<wire x1="17.018" y1="8.255" x2="17.145" y2="8.128" width="0.2032" layer="1"/>
-<via x="17.145" y="8.128" extent="1-16" drill="0.508"/>
-<wire x1="17.145" y1="8.128" x2="17.145" y2="6.35" width="0.2032" layer="16"/>
+<wire x1="14.82" y1="8.255" x2="15.748" y2="8.255" width="0.2032" layer="1"/>
+<wire x1="17.145" y1="7.112" x2="17.145" y2="6.35" width="0.2032" layer="16"/>
+<wire x1="15.748" y1="8.255" x2="16.764" y2="8.255" width="0.2032" layer="1"/>
+<via x="16.764" y="8.255" extent="1-16" drill="0.508"/>
+<wire x1="16.764" y1="8.255" x2="17.145" y2="7.874" width="0.2032" layer="16"/>
+<wire x1="17.145" y1="7.874" x2="17.145" y2="7.112" width="0.2032" layer="16"/>
 </signal>
 </signals>
