File: hardware/ISL29125 Breakout.sch (EAGLE design)
At the start: 16 parts, among them U1 ISL29125

Commit message: v01, revised after review, ready for protos
Parts:
- removed LOGO1: SFE_LOGO_NAME_FLAME.1_INCH, SparkFun-Aesthetics:SFE_LOGO_NAME_FLAME.1_INCH
- added LOGO2: SFE_LOGO_FLAME.2_INCH, SparkFun-Aesthetics:SFE_LOGO_FLAME.2_INCH
- added SJ2: (no value), SparkFun-Passives:SOLDERJUMPER_2WAYS
Connections:
- new net N$3: R2.2, SJ2.3
- new net N$4: R3.2, SJ2.1
- net 3.3V: now also SJ2.2; no longer R2.2, R3.2
Other:
- note added: "7bit: 0x44"
- note added: "I2C Address:"
- note added: "Read: 0x89"
- note added: "Write: 0x88"
Changed lines of the file:
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@@
 <part name="GND3" library="SparkFun-Aesthetics" deviceset="GND" device=""/>
 <part name="SUPPLY3" library="SparkFun-Aesthetics" deviceset="3.3V" device=""/>
-<part name="LOGO1" library="SparkFun-Aesthetics" deviceset="SFE_LOGO_NAME_FLAME" device=".1_INCH"/>
 <part name="LOGO3" library="SparkFun-Aesthetics" deviceset="OSHW-LOGO" device="S"/>
 <part name="FID1" library="SparkFun-Aesthetics" deviceset="FIDUCIAL" device="1X2"/>
@@
 <part name="STANDOFF2" library="SparkFun-Electromechanical" deviceset="STAND-OFF" device=""/>
 <part name="LOGO4" library="SparkFun-Aesthetics" deviceset="SFE_LOGO_FLAME" device=".2_INCH"/>
+<part name="SJ2" library="SparkFun-Passives" deviceset="SOLDERJUMPER_2WAY" device="S"/>
+<part name="SUPPLY4" library="SparkFun-Aesthetics" deviceset="3.3V" device=""/>
+<part name="LOGO2" library="SparkFun-Aesthetics" deviceset="SFE_LOGO_FLAME" device=".2_INCH"/>
 </parts>
 <sheets>
@@
 <text x="150.876" y="7.112" size="2.1844" layer="94">Jordan McConnell</text>
 <text x="238.252" y="7.112" size="2.1844" layer="94">v01</text>
+<text x="144.78" y="73.66" size="1.778" layer="97">7bit:    0x44</text>
+<text x="144.78" y="76.2" size="1.778" layer="97">I2C Address:</text>
+<text x="144.78" y="71.12" size="1.778" layer="97">Read: 0x89</text>
+<text x="144.78" y="68.58" size="1.778" layer="97">Write: 0x88</text>
 </plain>
 <instances>
@@
 <instance part="GND2" gate="1" x="76.2" y="78.74"/>
 <instance part="GND3" gate="1" x="109.22" y="76.2"/>
-<instance part="SUPPLY3" gate="G$1" x="162.56" y="114.3"/>
-<instance part="LOGO1" gate="G$1" x="157.48" y="33.02"/>
+<instance part="SUPPLY3" gate="G$1" x="160.02" y="124.46"/>
 <instance part="LOGO3" gate="G$1" x="233.68" y="45.72"/>
 <instance part="FID1" gate="G$1" x="246.38" y="25.4"/>
@@
 <instance part="STANDOFF2" gate="G$1" x="241.3" y="25.4"/>
 <instance part="LOGO4" gate="G$1" x="215.9" y="7.62"/>
+<instance part="SJ2" gate="G$1" x="160.02" y="116.84" rot="R270"/>
+<instance part="SUPPLY4" gate="G$1" x="172.72" y="111.76"/>
+<instance part="LOGO2" gate="G$1" x="205.74" y="7.62"/>
 </instances>
 <busses>
@@
 </segment>
 <segment>
-<pinref part="R2" gate="G$1" pin="2"/>
-<wire x1="157.48" y1="109.22" x2="157.48" y2="111.76" width="0.1524" layer="91"/>
-<wire x1="157.48" y1="111.76" x2="162.56" y2="111.76" width="0.1524" layer="91"/>
-<pinref part="R3" gate="G$1" pin="2"/>
-<wire x1="162.56" y1="111.76" x2="165.1" y2="111.76" width="0.1524" layer="91"/>
-<wire x1="165.1" y1="111.76" x2="165.1" y2="109.22" width="0.1524" layer="91"/>
-<wire x1="165.1" y1="111.76" x2="172.72" y2="111.76" width="0.1524" layer="91"/>
-<junction x="165.1" y="111.76"/>
 <pinref part="R4" gate="G$1" pin="2"/>
 <wire x1="172.72" y1="111.76" x2="172.72" y2="109.22" width="0.1524" layer="91"/>
+<pinref part="SUPPLY4" gate="G$1" pin="3.3V"/>
+</segment>
+<segment>
+<pinref part="SJ2" gate="G$1" pin="2"/>
 <pinref part="SUPPLY3" gate="G$1" pin="3.3V"/>
-<wire x1="162.56" y1="114.3" x2="162.56" y2="111.76" width="0.1524" layer="91"/>
-<junction x="162.56" y="111.76"/>
+<wire x1="160.02" y1="121.92" x2="160.02" y2="124.46" width="0.1524" layer="91"/>
 </segment>
 </net>
@@
 </segment>
 </net>
+<net name="N$3" class="0">
+<segment>
+<pinref part="R2" gate="G$1" pin="2"/>
+<wire x1="157.48" y1="109.22" x2="157.48" y2="111.76" width="0.1524" layer="91"/>
+<wire x1="157.48" y1="111.76" x2="152.4" y2="111.76" width="0.1524" layer="91"/>
+<wire x1="152.4" y1="111.76" x2="152.4" y2="116.84" width="0.1524" layer="91"/>
+<pinref part="SJ2" gate="G$1" pin="3"/>
+<wire x1="152.4" y1="116.84" x2="154.94" y2="116.84" width="0.1524" layer="91"/>
+</segment>
+</net>
+<net name="N$4" class="0">
+<segment>
+<pinref part="R3" gate="G$1" pin="2"/>
+<wire x1="165.1" y1="111.76" x2="165.1" y2="109.22" width="0.1524" layer="91"/>
+<wire x1="165.1" y1="111.76" x2="167.64" y2="111.76" width="0.1524" layer="91"/>
+<wire x1="167.64" y1="111.76" x2="167.64" y2="116.84" width="0.1524" layer="91"/>
+<pinref part="SJ2" gate="G$1" pin="1"/>
+<wire x1="167.64" y1="116.84" x2="165.1" y2="116.84" width="0.1524" layer="91"/>
+</segment>
+</net>

Commit message: hardware ready for reds, v10
Other:
- note added: "v10"
- note removed: "v01"
Changed lines of the file:
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@@
 <plain>
 <text x="150.876" y="7.112" size="2.1844" layer="94">Jordan McConnell</text>
-<text x="238.252" y="7.112" size="2.1844" layer="94">v01</text>
+<text x="238.252" y="7.112" size="2.1844" layer="94">v10</text>
 <text x="144.78" y="73.66" size="1.778" layer="97">7bit:    0x44</text>
 <text x="144.78" y="76.2" size="1.778" layer="97">I2C Address:</text>
